Commit message: new urdf xml

File: src/bxi_example_py_elf3/robot/elf3_lite/urdf/elf3_old.urdf (robot description, URDF)
Before this commit: robot elf3, 36 links, 35 joints
Links:
- removed link d435i_link
- removed link head_y_link
- removed link head_z_link
- removed link imu_link
- removed link mid360_link
- removed link torso_front_bottom_d435i_link
- link l_ankle_x_link: mass 0.37980156 -> 0.298065216713201
- link l_ankle_y_link: mass 0.01268984 -> 0.0126898593121342
- link l_elbow_y_link: mass 0.1020615 -> 0.0938669247468512
- link l_hip_x_link: mass 0.23202193 -> 0.214152254706427
- link l_hip_y_link: mass 1.74663835 -> 1.70384733340318
- link l_hip_z_link: mass 2.94332059 -> 2.84278184760334
- link l_knee_y_link: mass 1.86991215 -> 1.77390809
- link l_shoulder_x_link: mass 0.13939414 -> 0.130650985436178
- link l_shoulder_y_link: mass 0.99747353 -> 0.938482977144261
- link l_shoulder_z_link: mass 1.67349896 -> 1.29694131347632
- link l_wrist_x_link: mass 1.24945755 -> 0.65867493591403
- link l_wrist_y_link: mass 0.56828784 -> 0.243805170394381
- link l_wrist_z_link: mass 0.09977741 -> 0.106560860250811
- link r_ankle_x_link: mass 0.37980156 -> 0.298065216713202
- link r_ankle_y_link: mass 0.01268984 -> 0.0126898593121342
- link r_elbow_y_link: mass 0.1020615 -> 0.0938669107317605
- link r_hip_x_link: mass 0.23202193 -> 0.214152254706428
- link r_hip_y_link: mass 1.74663841 -> 1.70384734270319
- link r_hip_z_link: mass 2.94332069 -> 2.8427830619077
- link r_knee_y_link: mass 1.86991402 -> 1.77390996
- link r_shoulder_x_link: mass 0.13939414 -> 0.130650985436178
- link r_shoulder_y_link: mass 0.99747344 -> 0.938482977205647
- link r_shoulder_z_link: mass 1.67349843 -> 1.29694127388881
- link r_wrist_x_link: mass 1.24945755 -> 0.658674935909524
- link r_wrist_y_link: mass 0.56828784 -> 0.243805170389875
- link r_wrist_z_link: mass 0.09977741 -> 0.106560859874613
- link torso_link: mass 11.66386158 -> 12.004
- link waist_x_link: mass 0.24344947 -> 0.215642587680923
- link waist_y_link: mass 0.06620328 -> 0.0661517869264427
- link waist_z_link: mass 5.2693813 -> 4.95603362274037
Joints:
- removed joint d435i_joint
- removed joint head_y_joint
- removed joint head_z_joint
- removed joint imu_joint
- removed joint mid360_joint
- removed joint torso_front_bottom_d435i_joint
- joint l_ankle_x_joint: limit lower=-0.34907 upper=0.34907 effort=20 velocity=20 -> lower=-0.34907 upper=0.34907 effort=50 velocity=20
- joint l_elbow_y_joint: limit lower=-0.95993 upper=1.6581 effort=45 velocity=20 -> lower=-0.95993 upper=1.6581 effort=50 velocity=20
- joint l_hip_x_joint: limit lower=-0.48869 upper=3.0543 effort=150 velocity=20 -> lower=-0.48869 upper=3.0543 effort=100 velocity=20
- joint l_hip_y_joint: limit lower=-2.8798 upper=2.8798 effort=150 velocity=20 -> lower=-2.8798 upper=2.8798 effort=100 velocity=20
- joint l_hip_z_joint: limit lower=-2.8798 upper=2.8798 effort=45 velocity=20 -> lower=-2.8798 upper=2.8798 effort=50 velocity=20
- joint l_shoulder_x_joint: limit lower=-0.34907 upper=3.0543 effort=45 velocity=20 -> lower=-0.34907 upper=3.0543 effort=50 velocity=20
- joint l_shoulder_y_joint: limit lower=-2.8798 upper=2.8798 effort=45 velocity=20 -> lower=-2.8798 upper=2.8798 effort=50 velocity=20
- joint l_shoulder_z_joint: limit lower=-2.8798 upper=2.8798 effort=21 velocity=20 -> lower=-2.8798 upper=2.8798 effort=25 velocity=20
- joint l_wrist_x_joint: limit lower=-2.8798 upper=2.8798 effort=21 velocity=20 -> lower=-2.8798 upper=2.8798 effort=25 velocity=20
- joint l_wrist_y_joint: limit lower=-1.309 upper=1.309 effort=21 velocity=20 -> lower=-1.309 upper=1.309 effort=25 velocity=20
- joint l_wrist_z_joint: limit lower=-0.7854 upper=0.7854 effort=21 velocity=20 -> lower=-0.7854 upper=0.7854 effort=25 velocity=20
- joint r_ankle_x_joint: limit lower=-0.34907 upper=0.34907 effort=20 velocity=20 -> lower=-0.34907 upper=0.34907 effort=50 velocity=20
- joint r_elbow_y_joint: limit lower=-0.95993 upper=1.6581 effort=45 velocity=20 -> lower=-0.95993 upper=1.6581 effort=50 velocity=20
- joint r_hip_x_joint: limit lower=-3.0543 upper=0.48869 effort=150 velocity=20 -> lower=-3.0543 upper=0.48869 effort=100 velocity=20
- joint r_hip_y_joint: limit lower=-2.8798 upper=2.8798 effort=150 velocity=20 -> lower=-2.8798 upper=2.8798 effort=100 velocity=20
- joint r_hip_z_joint: limit lower=-2.8798 upper=2.8798 effort=45 velocity=20 -> lower=-2.8798 upper=2.8798 effort=50 velocity=20
- joint r_shoulder_x_joint: limit lower=-3.0543 upper=0.34907 effort=45 velocity=20 -> lower=-3.0543 upper=0.34907 effort=50 velocity=20
- joint r_shoulder_y_joint: limit lower=-2.8798 upper=2.8798 effort=45 velocity=20 -> lower=-2.8798 upper=2.8798 effort=50 velocity=20
- joint r_shoulder_z_joint: limit lower=-2.8798 upper=2.8798 effort=21 velocity=20 -> lower=-2.8798 upper=2.8798 effort=25 velocity=20
- joint r_wrist_x_joint: limit lower=-2.8798 upper=2.8798 effort=21 velocity=20 -> lower=-2.8798 upper=2.8798 effort=25 velocity=20
- joint r_wrist_y_joint: limit lower=-1.309 upper=1.309 effort=21 velocity=20 -> lower=-1.309 upper=1.309 effort=25 velocity=20
- joint r_wrist_z_joint: limit lower=-0.7854 upper=0.7854 effort=21 velocity=20 -> lower=-0.7854 upper=0.7854 effort=25 velocity=20
- joint waist_y_joint: limit lower=-0.5236 upper=0.5236 effort=90 velocity=20 -> lower=-0.5236 upper=0.5236 effort=100 velocity=20
- joint waist_z_joint: limit lower=-2.8798 upper=2.8798 effort=150 velocity=20 -> lower=-2.8798 upper=2.8798 effort=100 velocity=20

File: src/bxi_example_py_elf3/robot/elf3_lite/urdf/elf3_test1.urdf (robot description, URDF)
Before this commit: robot elf3, 36 links, 35 joints
Links:
- removed link d435i_link
- removed link head_y_link
- removed link head_z_link
- removed link imu_link
- removed link mid360_link
- removed link torso_front_bottom_d435i_link
- link l_ankle_x_link: mass 0.37980156 -> 0.298065216713201
- link l_ankle_y_link: mass 0.01268984 -> 0.0126898593121342
- link l_elbow_y_link: mass 0.1020615 -> 0.0938669247468512
- link l_hip_x_link: mass 0.23202193 -> 0.214152254706427
- link l_hip_y_link: mass 1.74663835 -> 1.70384733340318
- link l_hip_z_link: mass 2.94332059 -> 2.84278184760334
- link l_knee_y_link: mass 1.86991215 -> 1.77390809
- link l_shoulder_x_link: mass 0.13939414 -> 0.130650985436178
- link l_shoulder_y_link: mass 0.99747353 -> 0.938482977144261
- link l_shoulder_z_link: mass 1.67349896 -> 1.29694131347632
- link l_wrist_x_link: mass 1.24945755 -> 0.65867493591403
- link l_wrist_y_link: mass 0.56828784 -> 0.243805170394381
- link l_wrist_z_link: mass 0.09977741 -> 0.106560860250811
- link r_ankle_x_link: mass 0.37980156 -> 0.298065216713202
- link r_ankle_y_link: mass 0.01268984 -> 0.0126898593121342
- link r_elbow_y_link: mass 0.1020615 -> 0.0938669107317605
- link r_hip_x_link: mass 0.23202193 -> 0.214152254706428
- link r_hip_y_link: mass 1.74663841 -> 1.70384734270319
- link r_hip_z_link: mass 2.94332069 -> 2.8427830619077
- link r_knee_y_link: mass 1.86991402 -> 1.77390996
- link r_shoulder_x_link: mass 0.13939414 -> 0.130650985436178
- link r_shoulder_y_link: mass 0.99747344 -> 0.938482977205647
- link r_shoulder_z_link: mass 1.67349843 -> 1.29694127388881
- link r_wrist_x_link: mass 1.24945755 -> 0.658674935909524
- link r_wrist_y_link: mass 0.56828784 -> 0.243805170389875
- link r_wrist_z_link: mass 0.09977741 -> 0.106560859874613
- link torso_link: mass 11.66386158 -> 12.004
- link waist_x_link: mass 0.24344947 -> 0.215642587680923
- link waist_y_link: mass 0.06620328 -> 0.0661517869264427
- link waist_z_link: mass 5.2693813 -> 4.95603362274037
Joints:
- removed joint d435i_joint
- removed joint head_y_joint
- removed joint head_z_joint
- removed joint imu_joint
- removed joint mid360_joint
- removed joint torso_front_bottom_d435i_joint
- joint l_ankle_x_joint: limit lower=-0.34907 upper=0.34907 effort=20 velocity=20 -> lower=-0.34907 upper=0.34907 effort=50 velocity=20
- joint l_elbow_y_joint: limit lower=-0.95993 upper=1.6581 effort=45 velocity=20 -> lower=-0.95993 upper=1.6581 effort=50 velocity=20
- joint l_hip_x_joint: limit lower=-0.48869 upper=3.0543 effort=150 velocity=20 -> lower=-0.48869 upper=3.0543 effort=100 velocity=20
- joint l_hip_y_joint: limit lower=-2.8798 upper=2.8798 effort=150 velocity=20 -> lower=-2.8798 upper=2.8798 effort=100 velocity=20
- joint l_hip_z_joint: limit lower=-2.8798 upper=2.8798 effort=45 velocity=20 -> lower=-2.8798 upper=2.8798 effort=50 velocity=20
- joint l_knee_y_joint: origin xyz=0 0 -0.32 rpy=0 0 0 -> xyz=0 0 -0.38 rpy=0 0 0
- joint l_shoulder_x_joint: limit lower=-0.34907 upper=3.0543 effort=45 velocity=20 -> lower=-0.34907 upper=3.0543 effort=50 velocity=20
- joint l_shoulder_y_joint: limit lower=-2.8798 upper=2.8798 effort=45 velocity=20 -> lower=-2.8798 upper=2.8798 effort=50 velocity=20
- joint l_shoulder_z_joint: limit lower=-2.8798 upper=2.8798 effort=21 velocity=20 -> lower=-2.8798 upper=2.8798 effort=25 velocity=20
- joint l_wrist_x_joint: limit lower=-2.8798 upper=2.8798 effort=21 velocity=20 -> lower=-2.8798 upper=2.8798 effort=25 velocity=20
- joint l_wrist_y_joint: limit lower=-1.309 upper=1.309 effort=21 velocity=20 -> lower=-1.309 upper=1.309 effort=25 velocity=20
- joint l_wrist_z_joint: limit lower=-0.7854 upper=0.7854 effort=21 velocity=20 -> lower=-0.7854 upper=0.7854 effort=25 velocity=20
- joint r_ankle_x_joint: limit lower=-0.34907 upper=0.34907 effort=20 velocity=20 -> lower=-0.34907 upper=0.34907 effort=50 velocity=20
- joint r_elbow_y_joint: limit lower=-0.95993 upper=1.6581 effort=45 velocity=20 -> lower=-0.95993 upper=1.6581 effort=50 velocity=20
- joint r_hip_x_joint: limit lower=-3.0543 upper=0.48869 effort=150 velocity=20 -> lower=-3.0543 upper=0.48869 effort=100 velocity=20
- joint r_hip_y_joint: limit lower=-2.8798 upper=2.8798 effort=150 velocity=20 -> lower=-2.8798 upper=2.8798 effort=100 velocity=20
- joint r_hip_z_joint: limit lower=-2.8798 upper=2.8798 effort=45 velocity=20 -> lower=-2.8798 upper=2.8798 effort=50 velocity=20
- joint r_knee_y_joint: origin xyz=0 0 -0.32 rpy=0 0 0 -> xyz=0 0 -0.38 rpy=0 0 0
- joint r_shoulder_x_joint: limit lower=-3.0543 upper=0.34907 effort=45 velocity=20 -> lower=-3.0543 upper=0.34907 effort=50 velocity=20
- joint r_shoulder_y_joint: limit lower=-2.8798 upper=2.8798 effort=45 velocity=20 -> lower=-2.8798 upper=2.8798 effort=50 velocity=20
- joint r_shoulder_z_joint: limit lower=-2.8798 upper=2.8798 effort=21 velocity=20 -> lower=-2.8798 upper=2.8798 effort=25 velocity=20
- joint r_wrist_x_joint: limit lower=-2.8798 upper=2.8798 effort=21 velocity=20 -> lower=-2.8798 upper=2.8798 effort=25 velocity=20
- joint r_wrist_y_joint: limit lower=-1.309 upper=1.309 effort=21 velocity=20 -> lower=-1.309 upper=1.309 effort=25 velocity=20
- joint r_wrist_z_joint: limit lower=-0.7854 upper=0.7854 effort=21 velocity=20 -> lower=-0.7854 upper=0.7854 effort=25 velocity=20
- joint waist_y_joint: limit lower=-0.5236 upper=0.5236 effort=90 velocity=20 -> lower=-0.5236 upper=0.5236 effort=100 velocity=20
- joint waist_z_joint: limit lower=-2.8798 upper=2.8798 effort=150 velocity=20 -> lower=-2.8798 upper=2.8798 effort=100 velocity=20
